File: Entry/Entry-left.kicad_pcb (KiCad board)
At the start: 2 copper layers, 234.5 x 137.6 mm, 125 parts, among them U1 ProMicro, U2 PJ-320A

Commit message: Fix: draw both PCB outline & rename 1. rename project name from 'bottom-up' to 'Entry' 2. removed unused backup files 3. fix both PCB outline - margin 2.5mm, round 3mm 4. made gerber files
Parts:
- removed the REF** at (142.8, 98.1)
- removed the REF** at (22.0, 87.1)
- removed the REF** at (107.4, 76.9)
- removed the REF** at (248.6, 152.7)
- removed the REF** at (248.6, 87.1)
- removed the REF** at (175.1, 23.2)
- removed the REF** at (90.5, 44.5)
- removed the REF** at (22.0, 23.2)
- removed the REF** at (22.0, 152.7)
- removed the REF** at (90.1, 152.7)
- removed the REF** at (248.6, 23.2)
- removed the REF** at (90.1, 23.2)
- removed the REF** at (175.1, 152.7)
- added REF**: MountingHole_2.2mm_M2, MountingHole:MountingHole_2.2mm_M2, F.Cu at (39.0, 111.1)
- added REF**: MountingHole_2.2mm_M2, MountingHole:MountingHole_2.2mm_M2, F.Cu at (107.8, 78.3)
- added REF**: MountingHole_2.2mm_M2, MountingHole:MountingHole_2.2mm_M2, F.Cu at (27.4, 28.9)
- added REF**: MountingHole_2.2mm_M2, MountingHole:MountingHole_2.2mm_M2, F.Cu at (27.4, 147.0)
- added REF**: MountingHole_2.2mm_M2, MountingHole:MountingHole_2.2mm_M2, F.Cu at (250.2, 147.0)
- added REF**: MountingHole_2.2mm_M2, MountingHole:MountingHole_2.2mm_M2, F.Cu at (250.2, 28.9)
- moved D24 9.87 mm to (234.7, 43.7), turned to 0 degrees
- moved RESET1 8.09 mm to (84.0, 45.1)
- moved D54 4.07 mm to (249.1, 142.2)
- moved U2 2.21 mm to (253.2, 50.5)
- moved U1 1.73 mm to (43.8, 40.7)
- moved REF** 1.59 mm to (107.8, 116.4)
Routing:
- net row1: track 195.1 -> 183.0 mm
- net Net-(D24-A): track 6.08 -> 12.5 mm
- net RESET: track 45.7 -> 52.0 mm
- net GND: track 281.7 -> 286.7 mm
- net row6: track 369.4 -> 366.0 mm
- net col2: track 102.1 -> 98.8 mm
- net col5: track 182.0 -> 178.9 mm
- net col10: track 296.8 -> 293.8 mm
- net col11: track 297.1 -> 294.4 mm
- net col9: track 276.3 -> 273.9 mm
- net col7: track 182.7 -> 180.3 mm
- net col3: track 122.8 -> 120.4 mm
- net col6: track 216.7 -> 214.4 mm
- net col4: track 109.2 -> 106.9 mm
- net col8: track 258.9 -> 256.6 mm
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Other:
- board size 234.5 x 137.6 mm -> 228.8 x 124.1 mm
