File: Entry/Entry-right.kicad_pcb (KiCad board)
At the start: 2 copper layers, 103 parts, among them U1 ProMicro, U2 PJ-320A

Commit message: Fix: draw both PCB outline & rename 1. rename project name from 'bottom-up' to 'Entry' 2. removed unused backup files 3. fix both PCB outline - margin 2.5mm, round 3mm 4. made gerber files
Parts:
- added REF**: MountingHole_2.2mm_M2, MountingHole:MountingHole_2.2mm_M2, F.Cu at (32.2, 146.2)
- added REF**: MountingHole_2.2mm_M2, MountingHole:MountingHole_2.2mm_M2, F.Cu at (264.6, 146.2)
- added REF**: MountingHole_2.2mm_M2, MountingHole:MountingHole_2.2mm_M2, F.Cu at (203.2, 115.6)
- added REF**: MountingHole_2.2mm_M2, MountingHole:MountingHole_2.2mm_M2, F.Cu at (203.2, 77.5)
- added REF**: MountingHole_2.2mm_M2, MountingHole:MountingHole_2.2mm_M2, F.Cu at (32.2, 28.1)
- added REF**: MountingHole_2.2mm_M2, MountingHole:MountingHole_2.2mm_M2, F.Cu at (264.6, 28.1)
- moved D50 11.7 mm to (252.4, 142.8), turned to 0 degrees
- moved RESET1 5.88 mm to (208.0, 44.3), turned to 180 degrees
- moved U2 5.36 mm to (29.2, 49.7)
- moved U1 2.91 mm to (248.2, 39.9)
Connections:
- MX1 pad 1: unconnected-(MX1-COL-Pad1) -> col2
- MX10 pad 1: unconnected-(MX10-COL-Pad1) -> col5
- MX11 pad 1: unconnected-(MX11-COL-Pad1) -> col6
- MX12 pad 1: unconnected-(MX12-COL-Pad1) -> col7
- MX13 pad 1: unconnected-(MX13-COL-Pad1) -> col8
- MX14 pad 1: unconnected-(MX14-COL-Pad1) -> col1
- MX15 pad 1: unconnected-(MX15-COL-Pad1) -> col2
- MX16 pad 1: unconnected-(MX16-COL-Pad1) -> col3
- MX17 pad 1: unconnected-(MX17-COL-Pad1) -> col4
- MX18 pad 1: unconnected-(MX18-COL-Pad1) -> col5
- MX19 pad 1: unconnected-(MX19-COL-Pad1) -> col6
- MX2 pad 1: unconnected-(MX2-COL-Pad1) -> col3
- MX20 pad 1: unconnected-(MX20-COL-Pad1) -> col7
- MX21 pad 1: unconnected-(MX21-COL-Pad1) -> col8
- MX22 pad 1: unconnected-(MX22-COL-Pad1) -> col1
- MX23 pad 1: unconnected-(MX23-COL-Pad1) -> col2
- MX24 pad 1: unconnected-(MX24-COL-Pad1) -> col3
- MX25 pad 1: unconnected-(MX25-COL-Pad1) -> col4
- MX26 pad 1: unconnected-(MX26-COL-Pad1) -> col5
- MX27 pad 1: unconnected-(MX27-COL-Pad1) -> col6
- MX28 pad 1: unconnected-(MX28-COL-Pad1) -> col8
- MX29 pad 1: unconnected-(MX29-COL-Pad1) -> col1
- MX3 pad 1: unconnected-(MX3-COL-Pad1) -> col4
- MX30 pad 1: unconnected-(MX30-COL-Pad1) -> col2
- MX31 pad 1: unconnected-(MX31-COL-Pad1) -> col3
- MX32 pad 1: unconnected-(MX32-COL-Pad1) -> col4
- MX33 pad 1: unconnected-(MX33-COL-Pad1) -> col5
- MX34 pad 1: unconnected-(MX34-COL-Pad1) -> col6
- MX35 pad 1: unconnected-(MX35-COL-Pad1) -> col8
- MX36 pad 1: unconnected-(MX36-COL-Pad1) -> col1
- MX37 pad 1: unconnected-(MX37-COL-Pad1) -> col3
- MX38 pad 1: unconnected-(MX38-COL-Pad1) -> col6
- MX39 pad 1: unconnected-(MX39-COL-Pad1) -> col7
- MX4 pad 1: unconnected-(MX4-COL-Pad1) -> col5
- MX40 pad 1: unconnected-(MX40-COL-Pad1) -> col8
- MX41 pad 1: unconnected-(MX41-COL-Pad1) -> col9
- MX42 pad 1: unconnected-(MX42-COL-Pad1) -> col10
- MX43 pad 1: unconnected-(MX43-COL-Pad1) -> col11
- MX44 pad 1: unconnected-(MX44-COL-Pad1) -> col9
- MX45 pad 1: unconnected-(MX45-COL-Pad1) -> col10
- MX46 pad 1: unconnected-(MX46-COL-Pad1) -> col11
- MX47 pad 1: unconnected-(MX47-COL-Pad1) -> col10
- MX48 pad 1: unconnected-(MX48-COL-Pad1) -> col9
- MX49 pad 1: unconnected-(MX49-COL-Pad1) -> col10
- MX5 pad 1: unconnected-(MX5-COL-Pad1) -> col6
- MX50 pad 1: unconnected-(MX50-COL-Pad1) -> col11
- MX6 pad 1: unconnected-(MX6-COL-Pad1) -> col7
- MX7 pad 1: unconnected-(MX7-COL-Pad1) -> col2
- MX8 pad 1: unconnected-(MX8-COL-Pad1) -> col3
- MX9 pad 1: unconnected-(MX9-COL-Pad1) -> col4
- U1 pad 1: col1 -> col8
- U1 pad 10: row4 -> col6
- U1 pad 11: row5 -> col7
- U1 pad 12: row6 -> row1
- U1 pad 13: col11 -> row2
- U1 pad 14: col10 -> row3
- U1 pad 15: col9 -> row4
- U1 pad 16: col8 -> row5
- U1 pad 17: col7 -> row6
- U1 pad 18: col6 -> col9
- U1 pad 19: col5 -> col10
- U1 pad 2: col2 -> col1
- U1 pad 20: row1 -> col11
- U1 pad 5: col3 -> col2
- U1 pad 7: col4 -> col3
- U1 pad 8: row2 -> col4
- U1 pad 9: row3 -> col5
Routing:
- net col1: track 0.00 -> 323.0 mm, vias 0 -> 1
- net col2: track 0.00 -> 312.3 mm, vias 0 -> 1
- net col3: track 0.00 -> 306.8 mm, vias 0 -> 1
- net GND: track 0.00 -> 277.9 mm, vias 0 -> 1
- net col4: track 0.00 -> 265.4 mm, vias 0 -> 1
- net col5: track 0.00 -> 243.6 mm, vias 0 -> 1
- net VCC: track 0.00 -> 242.7 mm
- net col6: track 0.00 -> 241.2 mm, vias 0 -> 1
- net SCL: track 0.00 -> 231.3 mm
- net col7: track 0.00 -> 213.7 mm, vias 0 -> 1
- net col8: track 0.00 -> 203.4 mm, vias 0 -> 1
- net row6: track 195.2 -> 321.1 mm, vias 0 -> 1
- net col9: track 0.00 -> 122.2 mm
- net row5: track 199.0 -> 313.8 mm, vias 0 -> 1
- net col10: track 0.00 -> 105.8 mm
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Other:
- board outline added: 238.4 x 124.1 mm
